File: kicad/power.kicad_sch (KiCad schematic)
At the start: 99 parts, among them J1 12 V in (5.5x2.1), J2 TX power (shunt), U1 TPS54202DDCR, U2 TPS65131RGER, U3 TPS7A4701RGWR, U4 TPS7A3301RGWR, U5 LM2731XMF, U6 TLV75733PDBVR

Commit message: Optimized, costed BOM with LCSC numbers for every part
scripts/bom.py picks parts (Basic first, stock margin) and writes docs/bom.md,
fab/bom_jlcpcb.csv and scripts/parts.json; sch_lcsc.py fills LCSC fields from it.
Part changes: TPS7A4700RGWT for the out-of-stock TPS7A4701, BAV99 C2500, SS54 in SMA,
SMD1812P200TF16 polyfuse, 600R ferrite, Basic-value +5V/VDRV dividers (VDRV 15.4 V),
Sunlord SWPA6045 footprints, mic 100 nF C0G in 1206. AD7606C-16 and SPH0641 now
assembled by JLCPCB.
Parts:
- C1: LCSC TBD -> C294509
- C11, C12, C24, C25: LCSC TBD -> C380363
- C13, C2, C4, C5: LCSC TBD -> C14663
- C14: LCSC TBD -> C1679
- C15, C16, C21, C22, C23, C27: LCSC TBD -> C380364
- C17: LCSC TBD -> C53424
- C18: LCSC TBD -> C21120
- C19: LCSC TBD -> C57112
- C20: LCSC TBD -> C3904926
- C26, C28: LCSC TBD -> C388002
- C29: LCSC TBD -> C76599
- C3, C31, C33, C34: LCSC TBD -> C525507
- C30: LCSC TBD -> C55530
- C32: LCSC TBD -> C376771
- C35: LCSC TBD -> C970679
- C36, C38: LCSC TBD -> C15850
- C37: value 10u 16V X7R -> 10u 16V X7R 1206; footprint Capacitor_SMD:C_0805_2012Metric -> Capacitor_SMD:C_1206_3216Metric; LCSC TBD -> C380363
- C6, C7: LCSC TBD -> C12891
- C8: value 75p 50V C0G -> 100p 50V C0G; LCSC TBD -> C14858
- D1: footprint Diode_SMD:D_SMC -> Diode_SMD:D_SMA; LCSC TBD -> C22452
- D10, D11, D2, D3, D5, D7, D9: LCSC TBD -> C12624
- D4, D6, D8: LCSC TBD -> C2480
- F1: value 1812L200/16DR -> SMD1812P200TF16; LCSC TBD -> C20812
- FB1: value 220R@100MHz 0603 -> 600R@100MHz 0603; LCSC TBD -> C1002
- J1: LCSC TBD -> C22434582
- J2: LCSC TBD -> C492401
- JP1, JP2, JP3, JP4, JP5, JP6, TP1, TP10, TP11, TP2, TP3, TP4, TP5, TP6, TP7, TP8, TP9: LCSC TBD -> none (copper)
- L1: LCSC TBD -> C2041631
- L2, L3: footprint Inductor_SMD:L_Bourns_SRN6045TA -> Inductor_SMD:L_Sunlord_SWPA6045S; LCSC TBD -> C78804
- L4: footprint Inductor_SMD:L_Bourns_SRN6045TA -> Inductor_SMD:L_Sunlord_SWPA6045S; LCSC TBD -> C79272
- R1: LCSC TBD -> C25804
- R10, R13: LCSC TBD -> C22978
- R11: LCSC TBD -> C25821
- R12: LCSC TBD -> C48996814
- R14: LCSC TBD -> C23237
- R15: LCSC TBD -> C22961
- R16: LCSC TBD -> C23196
- R17: LCSC TBD -> C22807
- R18: value 13.3k 1% -> 13k 1%; LCSC TBD -> C22797
- R19: LCSC TBD -> C22809
- R2: value 511k 1% -> 510k 1%; LCSC TBD -> C23192
- R20, R21: LCSC TBD -> C21190
- R3: value 105k 1% -> 100k 1%; LCSC TBD -> C25803
- R4: value 100k 1% -> 75k 1%; LCSC TBD -> C23242
- R5: value 13.3k 1% -> 10k 1%; LCSC TBD -> C25804
- R6: LCSC TBD -> C4190
- R7: LCSC TBD -> C22775
- R8: LCSC TBD -> C321950
- R9: LCSC TBD -> C22795
- U1: LCSC TBD -> C191884
- U2: LCSC TBD -> C87663
- U3: value TPS7A4701RGWR -> TPS7A4700RGWT; LCSC TBD -> C28286
- U4: LCSC TBD -> C90082
- U5: LCSC TBD -> C485804
- U6: LCSC TBD -> C485517
Other:
- note added: "D. ANALOG RAILS: TPS7A4700 +5VA, TPS7A3301 -5VA (low noise, no LEDs)"
- note added: "Vout = 0.596 V x (1 + 75k/10k) = 5.07 V. EN UVLO about 7.3 V. Load about 1.4 A."
- note removed: "D. ANALOG RAILS: TPS7A4701 +5VA, TPS7A3301 -5VA (low noise, no LEDs)"
- note removed: "Vout = 0.596 V x (1 + 100k/13.3k) = 5.08 V. EN UVLO about 7 V. Load about 1.4 A."

Commit message: Switch to 16 x TLV320ADC5140, +3V3A rail, 3 A buck, datasheet library, transducer DNP
- ADC: 8 x AD7606C-16 ($470/board) -> 16 x TI TLV320ADC5140 at 192 kSPS ($50/board): TDM slave on a
  shared BCLK/FSYNC, I2C (SCL + 4 SDA groups), 2k/1k + 100 nF input network; project symbol from
  scripts/make_symbols.py; 9 clock buffers; J2 remapped
- power: +3V3A (second TPS7A4700, ANY-OUT 3.3 V); +5V buck TPS54202 -> TPS54302 (3 A), L1 10 uH 5 A
- checks and simulations updated for the new ADC input (all 18 checks and 10 sims pass)
- docs/datasheets: a PDF for every part, kept in step by scripts/datasheets.py (run by bom.py)
- design brief section 5a: interface bandwidth budget (no bus is a bottleneck; TX_EDGE = 1)
- CUSA-TR65 marked DNP for JLCPCB (hand-soldered), priced at DigiKey 100+
Parts:
- removed U1: TPS54202DDCR, Package_TO_SOT_SMD:SOT-23-6, symbol Regulator_Switching:TPS54202DDC
- added C39: 10u 25V X7R 1206, Capacitor_SMD:C_1206_3216Metric, symbol Device:C
- added C40, C41: 10u 16V X7R 1206, Capacitor_SMD:C_1206_3216Metric, symbol Device:C
- added C42: 1u 16V X7R, Capacitor_SMD:C_0603_1608Metric, symbol Device:C
- added JP7: cut to isolate, Jumper:SolderJumper-2_P1.3mm_Bridged_RoundedPad1.0x1.5mm, symbol Jumper:SolderJumper_2_Bridged
- added TP12: TP +3V3A, TestPoint:TestPoint_Pad_D1.5mm, symbol Connector:TestPoint
- added U1: TPS54302DDCR, Package_TO_SOT_SMD:SOT-23-6, symbol Regulator_Switching:TPS54302
- added U7: TPS7A4700RGWT, Package_DFN_QFN:Texas_RGW0020A_VQFN-20-1EP_5x5mm_P0.65mm_EP3.15x3.15mm_ThermalVias, symbol Regulator_Linear:TPS7A4701xRGW
- C20: LCSC C3904926 -> C2894191
- C30: LCSC C55530 -> C412624
- L1: value 15u Isat>=3.5A -> 10u Isat>=5A; LCSC C2041631 -> C2044906
Connections:
- net +5V: now also C39.1, U7.13 (EN), U7.15 (IN), U7.16 (IN)
- net BOOT_5V: now also U1.6 (BOOT)
- net EN_5V: now also U1.5 (EN)
- net FB_5V: now also U1.4 (FB)
- net GND: now also C39.2, C40.2, C41.2, C42.2, U1.1 (GND), U7.11 (0.2V), U7.12 (0.1V), U7.21 (EP), U7.7 (GND), U7.8 (1.6V)
- net SW_5V: now also U1.2 (SW)
- net VIN: now also U1.3 (VIN)
- new net +3V3A: JP7.2 (B), TP12.1
- new net 3V3A_REG: C40.1, C41.1, JP7.1 (A), U7.1 (OUT), U7.20 (OUT), U7.3 (SENSE/FB)
- new net NR_3V3A: C42.1, U7.14 (NR)
- no-connect marks 10 -> 15
Other:
- note added: "1.23 V x (1 + 150k/13k) = 15.4 V. Load, all 64 elements in CW at 40 kHz: about 0.24 A (sim/reports/tx_cw.md)."
- note added: "ANY-OUT 1.4 + 1.6 + 0.2 + 0.1 = 3.3 V. Load about 0.45 A (16 x TLV320ADC5140); 0.8 W in the LDO, thermal vias under the pad."
- note added: "B. +5V: TPS54302 buck (TI reference design), 3 A"
- note added: "I. +3V3A: TPS7A4700 low-noise LDO from +5V for the 16 ADCs' AVDD (analog rail: no LED)"
- note added: "Load < 0.15 A: ADC IOVDD, clock buffers, logic, mics."
- note added: "Load: 64 x OPA1678 (4 mA per channel): about 0.3 A on +5VA and on -5VA."
- note added: "Vout = 0.596 V x (1 + 75k/10k) = 5.07 V. EN UVLO about 7.3 V. Load about 1.6 A."
- note removed: "1.23 V x (1 + 150k/13.3k) = 15.1 V. Load, all 64 elements in CW at 40 kHz: about 0.24 A (sim/reports/tx_cw.md)."
- note removed: "B. +5V: TPS54202 buck (TI reference design), 2 A"
- note removed: "Load < 0.15 A: ADC VDRIVE, clock buffers, logic, mics."
- note removed: "Load: 64 x OPA1678 (4 mA per channel) + 8 x AD7606C AVCC: about 0.45 A on +5VA, 0.3 A on -5VA."
- note removed: "Vout = 0.596 V x (1 + 75k/10k) = 5.07 V. EN UVLO about 7.3 V. Load about 1.4 A."
- title: Power: 12 V in, +5V, +-6V5, +-5VA, VDRV, +3V3, 3V3_MIC -> Power: 12 V in, +5V, +-6V5, +-5VA, VDRV, +3V3, 3V3_MIC, +3V3A

Commit message: Board placement ready for routing; TPS26600 eFuse input protection
PCB (scripts/place.py builds kicad/aesa.kicad_pcb from the schematic, block by block):
- 192 x 301 mm, 4 layers (F.Cu / GND / GND / B.Cu), 3 mm corner bevels, parts >= 3 mm and copper
  >= 0.5 mm from the edge, 6 M3 holes, 3 fiducials
- all cables on the top edge: ribbon headers side by side in the middle, 12 V jack + eFuse top-left,
  +3V3A/+3V3 LDOs top-right; ADC blocks below; array; TX blocks; switchers at the bottom
- channels numbered down the columns: TX group k and ADC k sit under/over the column of CH 4k-3..4k,
  DRV lane left and RX lane right of each column on F.Cu (no crossings)
- hand templates from the mirrored pad positions (TX group, ADC, channel TX parts + op-amp, LM2731
  boost core); everything else placed by connectivity (switch loop first, decoupling at its pin)
- 2.5 mm soldering keep-out around transducer pads; silkscreen: block labels, test-point rail names,
  safety notes on the front
- scripts/placement_check.py: decoupling and switch-loop distances (all pass); DRC 0 violations

Schematic: TPS26600 eFuse (60 V / -60 V, off above 13.8 V and below 8.8 V, 1.6 A, auto-retry)
replaces the SS54 diode; polyfuse kept after it as back-up; test points for adapter voltage, input
current and fault. Array sheet grid follows the board's column-major numbering.
Parts:
- removed D1: SS54, Diode_SMD:D_SMA, symbol Device:D_Schottky
- added C43: 22n 50V X7R, Capacitor_SMD:C_0603_1608Metric, symbol Device:C
- added C44: 100n 50V X7R, Capacitor_SMD:C_0603_1608Metric, symbol Device:C
- added R22, R27: 100k 1%, Resistor_SMD:R_0603_1608Metric, symbol Device:R
- added R23: 5.6k 1%, Resistor_SMD:R_0603_1608Metric, symbol Device:R
- added R24: 10k 1%, Resistor_SMD:R_0603_1608Metric, symbol Device:R
- added R25: 7.5k 1%, Resistor_SMD:R_0603_1608Metric, symbol Device:R
- added R26: 15k 1%, Resistor_SMD:R_0603_1608Metric, symbol Device:R
- added TP13: TP VIN_JACK, TestPoint:TestPoint_Pad_D1.5mm, symbol Connector:TestPoint
- added TP14: TP IMON, TestPoint:TestPoint_Pad_D1.5mm, symbol Connector:TestPoint
- added TP15: TP FLT, TestPoint:TestPoint_Pad_D1.5mm, symbol Connector:TestPoint
- added U8: TPS26600PWPR, Package_SO:HTSSOP-16-1EP_4.4x5mm_P0.65mm_EP3.4x5mm_Mask2.66x2.46mm_ThermalVias, symbol Power_Management:TPS26600PWP
Connections:
- net VIN_FUSED is gone; now on net VIN: F1.2
- net GND: now also C43.2, C44.2, R24.2, R25.2, R26.2, U8.17 (RTN), U8.8 (RTN), U8.9 (GND)
- net VIN_JACK: now also C44.1, R22.1, R27.1, TP13.1, U8.1 (IN), U8.2 (IN); no longer F1.1
- new net EF_DVDT: C43.1, U8.12 (dVdT)
- new net EF_FLT: R27.2, TP15.1, U8.14 (~{FLT})
- new net EF_ILIM: R25.1, U8.11 (ILIM)
- new net EF_IMON: R26.1, TP14.1, U8.10 (IMON)
- new net EF_OVP: R23.2, R24.1, U8.5 (OVP)
- new net EF_UVLO: R22.2, R23.1, U8.3 (UVLO)
- new net VIN_PROT: F1.1, U8.15 (OUT), U8.16 (OUT)
- no-connect marks 15 -> 19
Other:
- note added: "A. 12 V INPUT: jack -> TPS26600 eFuse (resettable: auto-retry) -> polyfuse (back-up) -> VIN"
- note added: "UVLO/OVP divider 100k / 5.6k / 10k: on 8.8 V, off 13.8 V. ILIM 12 k/A -> 7.5 k = 1.6 A. dVdT 22 nF: 5 V/ms. IMON 72 uA/A into 15 k = 1.08 V/A (TP14). FLT low = fault (TP15)."
- note added: "eFuse: input rated 60 V and -60 V (reverse polarity), switches off above 13.8 V (protects the 14.5 V LM2731) and below 8.8 V, current limit 1.6 A."
- note removed: "A. 12 V INPUT: jack, polyfuse (16 V), SS54 reverse-polarity diode -> VIN"
- note removed: "Use a regulated 12 V adapter only (LM2731 VIN max 14 V). Jack 5.5 x 2.1 mm, >= 1.5 A."
