File: kicad/array.kicad_sch (KiCad schematic)
At the start: 0 parts

Commit message: Board placement ready for routing; TPS26600 eFuse input protection
PCB (scripts/place.py builds kicad/aesa.kicad_pcb from the schematic, block by block):
- 192 x 301 mm, 4 layers (F.Cu / GND / GND / B.Cu), 3 mm corner bevels, parts >= 3 mm and copper
  >= 0.5 mm from the edge, 6 M3 holes, 3 fiducials
- all cables on the top edge: ribbon headers side by side in the middle, 12 V jack + eFuse top-left,
  +3V3A/+3V3 LDOs top-right; ADC blocks below; array; TX blocks; switchers at the bottom
- channels numbered down the columns: TX group k and ADC k sit under/over the column of CH 4k-3..4k,
  DRV lane left and RX lane right of each column on F.Cu (no crossings)
- hand templates from the mirrored pad positions (TX group, ADC, channel TX parts + op-amp, LM2731
  boost core); everything else placed by connectivity (switch loop first, decoupling at its pin)
- 2.5 mm soldering keep-out around transducer pads; silkscreen: block labels, test-point rail names,
  safety notes on the front
- scripts/placement_check.py: decoupling and switch-loop distances (all pass); DRC 0 violations

Schematic: TPS26600 eFuse (60 V / -60 V, off above 13.8 V and below 8.8 V, 1.6 A, auto-retry)
replaces the SS54 diode; polyfuse kept after it as back-up; test points for adapter voltage, input
current and fault. Array sheet grid follows the board's column-major numbering.
Other:
- note added: "Transceiver array. Channel n = element n of the 8 x 8 grid, numbered down the columns (as on the board). Each channel takes DRVn from the TX drive and returns its amplified echo RXn to the ADCs."
- note removed: "Transceiver array. Channel n = element n of the 8 x 8 grid, row-major. Each channel takes DRVn from the TX drive and returns its amplified echo RXn to the ADCs."
