File: kicad/channel.kicad_sch (KiCad schematic)
At the start: 21 parts, among them U101 OPA1678IDR

Commit message: Block-first routing: all repeated blocks routed and passing, power input and +-6V5 hand-routed
Schematic
- TX groups and ADC inputs numbered in order (TXG01 = DRV1-4, ADC IN1..4 = RX1..4).
- Power sheets renumbered 1-8 with real references; eFuse RTN no longer tied to GND (TPS2660 9.3.5.5).
- Damped 100 uF bulk caps at the far ends of VIN (C50) and +5V (C51); header clock RC filters removed;
  switch-node snubbers kept as DNP footprints.

Layout and routing
- New routing toolchain: route.py (block stages), block_routes.py (hand-made block routes), maze.py
  (45-degree grid router with rip-up and a per-net time budget), route_lib.py (bend45, chamfer, copper
  checks), block_check.py (DRC and internal nets per block instance), board/cell views.
- Channel, ADC, TX group, clock buffer, enable buffer, mic and header blocks routed and passing
  block_check; no right-angle corners left.
- Designed TX control bus; SDI taps keep 0.7 mm from clock copper.
- Power: 12 V input (eFuse, RTN island, FLT via the front copper) and TPS65131 +-6V5 section with fixed
  templates and hand routing; each power section counts as its own block; the +3V3 LED overflows into
  the gap beside its section.

docs/routing_and_emi.md describes the routing and EMI rules; sim/mic_clock_si adds the mic clock check.
Connections:
- net FB1: now also U101.6 (-); no longer U101.2 (-)
- net GND: now also U101.3 (+); no longer U101.5 (+)
- net INV2: now also U101.2 (-); no longer U101.6 (-)
- net LIM: now also U101.5 (+); no longer U101.3 (+)
- net OUT2: now also U101.1; no longer U101.7
- net S1: now also U101.7; no longer U101.1
