File: kicad/clk_buf.kicad_sch (KiCad schematic)
At the start: 5 parts, among them U1 74LVC2G34

Commit message: Block-diagram top page, power review fixes, readable sheets
Top level
- Page 1 is now a block diagram of the signal flow (FPGA -> headers ->
  clock buffers / TX drive -> transceivers -> ADCs -> FPGA, mics, power).
- New group sheets hold the reused cells: tx (16 tx_group + 4 en_buf),
  array (64 channel), adcs (8 adc), mics (8 mic), clocks (7 clk_buf).
  Power and headers stay directly under the top. All written by gen_top.py,
  which now also survives a kicad-cli re-save of a cell sheet.

Power (review findings)
- Polyfuse 1812L200/16DR (16 V), TPS65131RGER stated explicitly, input caps
  2 x 10u 1206, 50 V caps on 12 V, inductor values carry minimum Isat.
- +3V3: TLV75733P (ceramic-stable) replaces TLV1117-33.
- New JP5/JP6 isolate +-6V5; every rail: REG node -> jumper -> rail with TP,
  LED (not on analog LDOs) and PWR_FLAG.
- Power sheet is now generated by build_cells.py in a 2x3 block layout
  (build_power.py removed).

Readability and small fixes
- Rails on sideways pins use labelled flags; sideways GND symbols hide text.
- tx_group: 595 outputs wired straight to the drivers.
- Title blocks on every sheet; channel sheet notes and field placement fixed
  (sch_fields.py --only, sch_annotate.py).
- ADC_SDI 10k pull-down, ADC reset/DOUT notes, mic cap 50 V.
- ERC 0 violations, 1,704 parts. PDFs: docs/schematics/00..13.
Other:
- company: (none) -> Hybrid 8x8 ultrasonic AESA
- title: (none) -> Clock buffer (x7): 74LVC2G34, 33 R outputs

Commit message: Optimized, costed BOM with LCSC numbers for every part
scripts/bom.py picks parts (Basic first, stock margin) and writes docs/bom.md,
fab/bom_jlcpcb.csv and scripts/parts.json; sch_lcsc.py fills LCSC fields from it.
Part changes: TPS7A4700RGWT for the out-of-stock TPS7A4701, BAV99 C2500, SS54 in SMA,
SMD1812P200TF16 polyfuse, 600R ferrite, Basic-value +5V/VDRV dividers (VDRV 15.4 V),
Sunlord SWPA6045 footprints, mic 100 nF C0G in 1206. AD7606C-16 and SPH0641 now
assembled by JLCPCB.
Parts:
- C1: LCSC TBD -> C14663
- R1, R2: LCSC TBD -> C23140
- R3: LCSC TBD -> C25803
- U1: LCSC TBD -> C52140488

Commit message: Switch to 16 x TLV320ADC5140, +3V3A rail, 3 A buck, datasheet library, transducer DNP
- ADC: 8 x AD7606C-16 ($470/board) -> 16 x TI TLV320ADC5140 at 192 kSPS ($50/board): TDM slave on a
  shared BCLK/FSYNC, I2C (SCL + 4 SDA groups), 2k/1k + 100 nF input network; project symbol from
  scripts/make_symbols.py; 9 clock buffers; J2 remapped
- power: +3V3A (second TPS7A4700, ANY-OUT 3.3 V); +5V buck TPS54202 -> TPS54302 (3 A), L1 10 uH 5 A
- checks and simulations updated for the new ADC input (all 18 checks and 10 sims pass)
- docs/datasheets: a PDF for every part, kept in step by scripts/datasheets.py (run by bom.py)
- design brief section 5a: interface bandwidth budget (no bus is a bottleneck; TX_EDGE = 1)
- CUSA-TR65 marked DNP for JLCPCB (hand-soldered), priced at DigiKey 100+
Other:
- title: Clock buffer (x7): 74LVC2G34, 33 R outputs -> Clock buffer (x9): 74LVC2G34, 33 R outputs

Commit message: Block-first routing: all repeated blocks routed and passing, power input and +-6V5 hand-routed
Schematic
- TX groups and ADC inputs numbered in order (TXG01 = DRV1-4, ADC IN1..4 = RX1..4).
- Power sheets renumbered 1-8 with real references; eFuse RTN no longer tied to GND (TPS2660 9.3.5.5).
- Damped 100 uF bulk caps at the far ends of VIN (C50) and +5V (C51); header clock RC filters removed;
  switch-node snubbers kept as DNP footprints.

Layout and routing
- New routing toolchain: route.py (block stages), block_routes.py (hand-made block routes), maze.py
  (45-degree grid router with rip-up and a per-net time budget), route_lib.py (bend45, chamfer, copper
  checks), block_check.py (DRC and internal nets per block instance), board/cell views.
- Channel, ADC, TX group, clock buffer, enable buffer, mic and header blocks routed and passing
  block_check; no right-angle corners left.
- Designed TX control bus; SDI taps keep 0.7 mm from clock copper.
- Power: 12 V input (eFuse, RTN island, FLT via the front copper) and TPS65131 +-6V5 section with fixed
  templates and hand routing; each power section counts as its own block; the +3V3 LED overflows into
  the gap beside its section.

docs/routing_and_emi.md describes the routing and EMI rules; sim/mic_clock_si adds the mic clock check.
Parts:
- R1, R2: value 33 1% -> 47 1%; LCSC C23140 -> C23182
Other:
- note added: "Clock fan-out: 74LVC2G34, both gates on IN, 47 R series termination per output (with the ~20 R driver: matches the 61 ohm 0.25 mm clock traces)"
- note added: "Each output drives at most 4 loads, clustered at the far end of its trace (series termination needs that: sim/reports/mic_clock_si.md)."
- note removed: "Clock fan-out: 74LVC2G34 at the header, both gates on IN, 33 R series termination per output"
- note removed: "Each output drives at most 4 loads (series termination works for a lumped load at the far end)."
- title: Clock buffer (x9): 74LVC2G34, 33 R outputs -> Clock buffer (x10): 74LVC2G34, 47 R outputs
