File: kicad/mics.kicad_sch (KiCad schematic)
At the start: 0 parts

Commit message: Block-first routing: all repeated blocks routed and passing, power input and +-6V5 hand-routed
Schematic
- TX groups and ADC inputs numbered in order (TXG01 = DRV1-4, ADC IN1..4 = RX1..4).
- Power sheets renumbered 1-8 with real references; eFuse RTN no longer tied to GND (TPS2660 9.3.5.5).
- Damped 100 uF bulk caps at the far ends of VIN (C50) and +5V (C51); header clock RC filters removed;
  switch-node snubbers kept as DNP footprints.

Layout and routing
- New routing toolchain: route.py (block stages), block_routes.py (hand-made block routes), maze.py
  (45-degree grid router with rip-up and a per-net time budget), route_lib.py (bend45, chamfer, copper
  checks), block_check.py (DRC and internal nets per block instance), board/cell views.
- Channel, ADC, TX group, clock buffer, enable buffer, mic and header blocks routed and passing
  block_check; no right-angle corners left.
- Designed TX control bus; SDI taps keep 0.7 mm from clock copper.
- Power: 12 V input (eFuse, RTN island, FLT via the front copper) and TPS65131 +-6V5 section with fixed
  templates and hand routing; each power section counts as its own block; the +3V3 LED overflows into
  the gap beside its section.

docs/routing_and_emi.md describes the routing and EMI rules; sim/mic_clock_si adds the mic clock check.
Other:
- note added: "MEMS mics. Mics 2k-1 and 2k share MIC_DATAk-1 (SEL high on the odd one). One clock per mic pair: MIC_CLK_A mics 1-2, B 3-4, C 5-6, D 7-8."
- note removed: "MEMS mics. Mics 2k-1 and 2k share MIC_DATAk-1 (SEL high on the odd one). MIC_CLK_A feeds mics 1-4, MIC_CLK_B mics 5-8."
Changed lines of the file:
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@@
 		(company "Hybrid 8x8 ultrasonic AESA")
 	)
-	(text "MEMS mics. Mics 2k-1 and 2k share MIC_DATAk-1 (SEL high on the odd one). MIC_CLK_A feeds mics 1-4, MIC_CLK_B mics 5-8."
+	(text "MEMS mics. Mics 2k-1 and 2k share MIC_DATAk-1 (SEL high on the odd one). One clock per mic pair: MIC_CLK_A mics 1-2, B 3-4, C 5-6, D 7-8."
 		(exclude_from_sim no)
 		(at 38.10 30.48 0)
@@
 			(project "aesa"
 				(path "/35d88121-1d5f-4a62-9009-788ea6bf93dd/f773ca19-03bb-5251-9781-0307c4b28445"
-					(page "117")
+					(page "118")
 				)
 			)
@@
 			(project "aesa"
 				(path "/35d88121-1d5f-4a62-9009-788ea6bf93dd/f773ca19-03bb-5251-9781-0307c4b28445"
-					(page "118")
+					(page "119")
 				)
 			)
@@
 		)
 	)
-	(global_label "MIC_CLK_A"
+	(global_label "MIC_CLK_B"
 		(shape passive)
 		(at 231.14 53.34 180)
@@
 			(project "aesa"
 				(path "/35d88121-1d5f-4a62-9009-788ea6bf93dd/f773ca19-03bb-5251-9781-0307c4b28445"
-					(page "119")
+					(page "120")
 				)
 			)
@@
 		)
 	)
-	(global_label "MIC_CLK_A"
+	(global_label "MIC_CLK_B"
 		(shape passive)
 		(at 322.58 53.34 180)
@@
 			(project "aesa"
 				(path "/35d88121-1d5f-4a62-9009-788ea6bf93dd/f773ca19-03bb-5251-9781-0307c4b28445"
-					(page "120")
+					(page "121")
 				)
 			)
@@
 		)
 	)
-	(global_label "MIC_CLK_B"
+	(global_label "MIC_CLK_C"
 		(shape passive)
 		(at 48.26 86.36 180)
@@
 			(project "aesa"
 				(path "/35d88121-1d5f-4a62-9009-788ea6bf93dd/f773ca19-03bb-5251-9781-0307c4b28445"
-					(page "121")
+					(page "122")
 				)
 			)
@@
 		)
 	)
-	(global_label "MIC_CLK_B"
+	(global_label "MIC_CLK_C"
 		(shape passive)
 		(at 139.70 86.36 180)
@@
 			(project "aesa"
 				(path "/35d88121-1d5f-4a62-9009-788ea6bf93dd/f773ca19-03bb-5251-9781-0307c4b28445"
-					(page "122")
+					(page "123")
 				)
 			)
@@
 		)
 	)
-	(global_label "MIC_CLK_B"
+	(global_label "MIC_CLK_D"
 		(shape passive)
 		(at 231.14 86.36 180)
@@
 			(project "aesa"
 				(path "/35d88121-1d5f-4a62-9009-788ea6bf93dd/f773ca19-03bb-5251-9781-0307c4b28445"
-					(page "123")
+					(page "124")
 				)
 			)
@@
 		)
 	)
-	(global_label "MIC_CLK_B"
+	(global_label "MIC_CLK_D"
 		(shape passive)
 		(at 322.58 86.36 180)
@@
 			(project "aesa"
 				(path "/35d88121-1d5f-4a62-9009-788ea6bf93dd/f773ca19-03bb-5251-9781-0307c4b28445"
-					(page "124")
-				)
-			)
+					(page "125")
+				)
+			)
