File: kicad/power_analog.kicad_sch (KiCad schematic)
At the start: 53 parts, among them U2 TPS65131RGER, U3 TPS7A4700RGWT, U4 TPS7A3301RGWR, U7 TPS7A4700RGWT

Commit message: Block-first routing: all repeated blocks routed and passing, power input and +-6V5 hand-routed
Schematic
- TX groups and ADC inputs numbered in order (TXG01 = DRV1-4, ADC IN1..4 = RX1..4).
- Power sheets renumbered 1-8 with real references; eFuse RTN no longer tied to GND (TPS2660 9.3.5.5).
- Damped 100 uF bulk caps at the far ends of VIN (C50) and +5V (C51); header clock RC filters removed;
  switch-node snubbers kept as DNP footprints.

Layout and routing
- New routing toolchain: route.py (block stages), block_routes.py (hand-made block routes), maze.py
  (45-degree grid router with rip-up and a per-net time budget), route_lib.py (bend45, chamfer, copper
  checks), block_check.py (DRC and internal nets per block instance), board/cell views.
- Channel, ADC, TX group, clock buffer, enable buffer, mic and header blocks routed and passing
  block_check; no right-angle corners left.
- Designed TX control bus; SDI taps keep 0.7 mm from clock copper.
- Power: 12 V input (eFuse, RTN island, FLT via the front copper) and TPS65131 +-6V5 section with fixed
  templates and hand routing; each power section counts as its own block; the +3V3 LED overflows into
  the gap beside its section.

docs/routing_and_emi.md describes the routing and EMI rules; sim/mic_clock_si adds the mic clock check.
Parts:
- added C47, C48: 470p 50V C0G DNP, Capacitor_SMD:C_0603_1608Metric, symbol Device:C
- added R29, R30: 4.7 1% DNP, Resistor_SMD:R_0603_1608Metric, symbol Device:R
- C20: LCSC C2894191 -> C3904926
- R14: LCSC C23237 -> C321989
Connections:
- net GND: now also C47.2, C48.2
- net SW_N: now also R30.1
- net SW_P: now also R29.1
- new net: C47.1, R29.2
- new net: C48.1, R30.2
Other:
- note added: "(low = eFuse fault)."
- note added: "+-5VA (receivers)."
- note added: "+6V5 = 1.213 V x (1 + 562k/130k) = 6.46 V (R9508 / R9509). -6V5 = -1.213 V x 649k/121k = -6.51 V (R9511 / R9512)."
- note added: "-> VDRV."
- note added: "1. 12 V jack J9501 -> eFuse U9508 -> F9501 -> VIN."
- note added: "2. VIN -> buck U9501 -> +5V. 4. VIN -> boost U9505"
- note added: "3. +5V -> LDO U9506 -> +3V3 -> 5. FB9501 -> 3V3_MIC."
- note added: "3V3_MIC) and the ground test points. Power 2:"
- note added: "6. +-6V5: TPS65131RGER U9502, boost + inverter from +5V (feeds the analog LDOs only)"
- note added: "6. +5V -> U9502 -> +-6V5 -> 7. LDOs U9503 / U9504 ->"
- note added: "7. +-5VA: low-noise LDOs TPS7A4700 U9503 / TPS7A3301 U9504"
- note added: "8. +3V3A: TPS7A4700 low-noise LDO U9507 from +5V"
- note added: "8. +5V -> LDO U9507 -> +3V3A (ADC AVDD)."
- note added: "DNP (fit only if a switch node rings)."
- note added: "Drawn with the pin-identical TPS65130 symbol: order TPS65131RGER (2 A switches). PSP/PSN low: fixed-frequency PWM. R9529 + C9547 and R9530 + C9548: switch-node snubbers,"
- note added: "First power-up: J9502 shunt off, bench supply 12 V"
- note added: "IMON (TP9514) 1.08 V per A in. FLT (TP9515) high"
- note added: "Power 1: sections 1-5 (input, +5V, +3V3, VDRV,"
- note added: "Then fit the J9502 shunt: VDRV 15.4 V."
- note added: "sections 6-8 (+-6V5, +-5VA, +3V3A)."
- note removed: "+5V -> U2 -> +-6V5 -> U3 / U4 -> +-5VA (receivers)."
- note removed: "+5V -> U6 -> +3V3 -> FB1 -> 3V3_MIC."
- note removed: "+5V -> U7 -> +3V3A (ADC AVDD)."
- note removed: "+6V5 = 1.213 V x (1 + 562k/130k) = 6.46 V. -6V5 = -1.213 V x 649k/121k = -6.51 V."
- note removed: "12 V jack -> eFuse U8 -> F1 -> VIN."
- note removed: "C. +-6V5: TPS65131RGER boost + inverter from +5V (feeds the analog LDOs only)"
- note removed: "D. +-5VA: TPS7A4700 / TPS7A3301 low-noise LDOs"
- note removed: "Drawn with the pin-identical TPS65130 symbol: order TPS65131RGER (2 A switches). PSP/PSN low: fixed-frequency PWM."
- note removed: "First power-up: J2 shunt off, bench supply 12 V"
- note removed: "G ground. Power 2: C +-6V5, D +-5VA, I +3V3A."
- note removed: "I. +3V3A: TPS7A4700 low-noise LDO from +5V"
- note removed: "IMON 1.08 V per A in. FLT high (low = eFuse fault)."
- note removed: "Power 1: A input, B +5V, E VDRV, F +3V3, H 3V3_MIC,"
- note removed: "Then fit J2: VDRV 15.4 V."
- note removed: "VIN -> U1 buck -> +5V. VIN -> U5 boost -> VDRV."
